File: signal_power_filter.kicad_sch (KiCad schematic)
At the start: 23 parts, among them J1 Barrel_Jack, J2 Guitar Jack, U1 LM7812_TO220, U2 LM7912_TO220

Commit message: began layout
Parts:
- J1: value Barrel_Jack -> PWR_IN
- U1, U2: footprint Package_TO_SOT_THT:TO-220-3_Vertical -> Package_TO_SOT_THT:TO-220-3_Horizontal_TabDown
Connections:
- net GND: now also J2.1; no longer J2.S
- net at R4.1: now also J2.2; no longer J2.T
Changed lines of the file:
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@@
 			)
 		)
-		(property "Value" "Barrel_Jack"
+		(property "Value" "PWR_IN"
 			(at 69.596 26.162 0)
 			(effects
@@
 			)
 		)
-		(pin "S"
-		)
-		(pin "T"
+		(pin "2"
+		)
+		(pin "1"
 		)
 		(instances
@@
 			)
 		)
-		(property "Footprint" "Package_TO_SOT_THT:TO-220-3_Vertical"
+		(property "Footprint" "Package_TO_SOT_THT:TO-220-3_Horizontal_TabDown"
 			(at 219.71 39.37 0)
 			(effects
@@
 			)
 		)
-		(property "Footprint" "Package_TO_SOT_THT:TO-220-3_Vertical"
+		(property "Footprint" "Package_TO_SOT_THT:TO-220-3_Horizontal_TabDown"
 			(at 189.23 29.845 0)
 			(effects
