File: DronePedal.kicad_pcb (KiCad board)
At the start: 2 copper layers, 177.8 x 152.4 mm, 453 parts, among them J1 Barrel_Jack, J2 Guitar Jack, J3 SIG_OUT, Q1 BC550, Q10 BC550, Q11 BC550, Q12 BC550, Q13 BC550, Q14 BC550, Q15 BC550, Q16 BC550, Q17 BC550, Q18 BC550, Q19 BC550, Q2 BC550, Q20 BC550, Q21 BC550, Q22 BC550, Q23 BC550, Q24 BC550, Q25 BC550, Q26 BC550, Q27 BC550, Q28 BC550, Q29 BC550, Q3 BC550, Q30 BC550, Q31 BC550, Q32 BC550, Q33 BC550, Q4 BC550, Q5 BC550, Q6 BC550, Q7 BC550, Q8 BC550, Q9 BC550, SW10 SW_SPST, SW11 SW_SPST, SW12 SW_SP4T, SW13 SW_SPST, SW14 SW_SPST, SW15 SW_SPST, SW16 SW_SPST, SW17 SW_SPST, SW18 SW_SPST, SW19 SW_SPST, SW2 SW_SPST, SW20 SW_SP4T, SW21 SW_SPST, SW22 SW_SPST, SW23 SW_SPST, SW24 SW_SPST, SW25 SW_SPST, SW3 SW_SPST, SW4 SW_SP4T, SW5 SW_SPST, SW6 SW_SPST, SW7 SW_SPST, SW8 SW_SPST, SW9 SW_SPST, U1 LM7812_TO220, U10 TL072, U11 TL074, U12 TL072, U13 TL072, U14 TL072, U15 TL074, U2 LM7912_TO220, U3 TL072, U4 TL072, U5 TL072, U6 TL074, U7 TL072, U8 TL072, U9 TL072

Commit message: began layout
Parts:
- J1: value Barrel_Jack -> PWR_IN
- U1, U2: footprint Package_TO_SOT_THT:TO-220-3_Vertical -> Package_TO_SOT_THT:TO-220-3_Horizontal_TabDown
- moved C26 439.3 mm to (416.2, 294.1)
- moved C27 439.3 mm to (416.2, 298.1)
- moved C28 439.3 mm to (416.2, 302.1)
- moved C29 439.3 mm to (416.2, 306.2)
- moved J3 439.3 mm to (420.5, 269.7)
- moved R62 427.9 mm to (470.5, 323.6)
- moved SW15 391.5 mm to (310.8, -132.6)
- moved RV11 386.8 mm to (435.1, 349.4)
- moved RV12 386.8 mm to (435.1, 353.5)
- moved RV13 386.8 mm to (435.1, 357.6)
- moved RV14 386.8 mm to (435.1, 361.6)
- moved RV16 386.8 mm to (448.4, 329.2)
- moved RV17 386.8 mm to (448.4, 333.2)
- moved RV18 386.8 mm to (448.4, 337.3)
- moved RV19 386.8 mm to (448.4, 341.4)
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Connections:
- J2 pad 1: (no net) -> GND
- J2 pad 2: (no net) -> Net-(J2-Pad2)
- R4 pad 1: Net-(J2-PadT) -> Net-(J2-Pad2)
Routing:
- net Net-(U4A--): track 0.00 -> 17.8 mm
- net Net-(R16-Pad2): track 0.00 -> 15.1 mm
- net Net-(R23-Pad1): track 0.00 -> 5.46 mm
- net Net-(R19-Pad1): track 0.00 -> 3.63 mm
- net Net-(U4B--): track 0.00 -> 2.69 mm
- net -12V: track 0.00 -> 2.27 mm
- net +12V: track 0.00 -> 2.26 mm
- added copper zone on B.Cu, net GND
- added copper zone on F.Cu, net GND

Commit message: more routing progress made
Parts:
- moved R62 441.0 mm to (94.1, 93.8)
- moved RV5 432.6 mm to (61.0, 108.0)
- moved RV6 407.8 mm to (100.1, 96.8), turned to -90 degrees
- moved R60 407.7 mm to (58.4, 105.0)
- moved R59 407.3 mm to (58.4, 102.8)
- moved R61 401.6 mm to (64.0, 110.7), turned to -90 degrees
- moved RV9 400.8 mm to (116.8, 97.8), turned to 90 degrees
- moved RV7 393.6 mm to (105.7, 117.9)
- moved R63 382.2 mm to (99.2, 91.5), turned to 180 degrees
- moved R64 376.2 mm to (102.5, 101.0), turned to -90 degrees
- moved R70 376.1 mm to (114.3, 100.8)
- moved R65 372.7 mm to (100.3, 115.1), turned to -90 degrees
- moved R68 371.4 mm to (114.3, 103.2)
- moved R66 371.3 mm to (102.6, 117.1), turned to -90 degrees
- moved R67 365.8 mm to (108.7, 120.4), turned to -90 degrees
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